File: kicad/RF_Frontend.kicad_sch (KiCad schematic)
At the start: 13 parts, among them J1 Conn_Coaxial, U1 AD8317

Commit message: Add calibration scripts, documentation, simulation tools, and KiCad updates
- cal/calibration.py: 3-phase RF linearity calibration (29 freq, 28 power steps,
  1 MHz–10 GHz, direct generator→DUT, no attenuator, NRP sensor 0.01 dBm precision)
- cal/temp_calibration.py: temperature calibration via Vötsch chamber (16–40°C,
  Vötsch SIMSERV TCP driver, tracking generator source, outputs TEMP_COEFF_DB_PER_C[])
- cal/results/: dry-run calibration tables (.h/.json), figures, PDF reports
- doc/: ADC signal path analysis, calibration procedure (3-phase), lab optimisation
  guide updated for 1 MHz–10 GHz range and temperature correction firmware formula
- doc/diagrams/: PlantUML/Mermaid source + rendered PNGs for pipeline, firmware,
  and RF signal chain architectures
- sim/ltpwr_to_touchstone.py: LTpowerAnalyzer Z(f) → Touchstone S1P + Z1P via
  scikit-rf for SIwave PI-AC Decoupling Optimization DC/DC source impedance import
- sim/Measured_source_impedance.txt/.s1p/.z1p: DC/DC output impedance measurement
  and converted Touchstone files (100 Hz–10 MHz, 201 points)
- kicad/: updated schematics (MCU, power management, RF frontend, UI) and PCB layout
- kicad/fixture-rev_A/: test fixture DXF drawings
- lib/: Würth 744231091 datasheet, Hammond 1590A board outline footprint
- pp_3d_printer_setup_spec.md, pp_horn_antenna_manufacturing_spec.md: process specs

Co-Authored-By: Claude Sonnet 4.6 <noreply@anthropic.com>
Parts:
- C3: value 1nF -> 1nF / C0G
- C6: value 8.2pF -> 8.2pF / C0G
- R4: value 100R -> 1k; now not fitted
- R5: value 0R -> 12k
Other:
- moved on the sheet: C1, C2, C3, C4, C5, C6, J1, R1, R2, R3, R5, U1
