File: kicad/RF_Frontend.kicad_sch (KiCad schematic)
At the start: 13 parts, among them J1 Conn_Coaxial, U1 AD8317

Commit message: Use Würth 60312202114307 SMA connector
Replace J1 with the shorter Würth WR-SMA connector, add its footprint and 3D model, make KiCad library paths portable, and include the reviewed EMerge geometry/export updates. Generated results and private local paths are intentionally excluded.
Parts:
- removed J1: Conn_Coaxial, Connector_Coaxial:SMA_Amphenol_132289_EdgeMount, symbol Connector:Conn_Coaxial
- added J1: 60312202114307, Connector_SMD_Wurth:J_Wurth_WR-SMA_60312202114307, symbol Wurth:60312202114307
- C4: LCSC (none) -> C9900014224; TME (none) -> AC0402KRX7R7BB104
- C5: footprint Capacitor_SMD:C_0201_0603Metric -> Capacitor_SMD:C_0805_2012Metric
- R3: LCSC (none) -> C9900199398; TME (none) -> RC0402JR-071K8
Connections:
- net GND: now also J1.2 (Ext)
- net at C1.1, R1.1, R2.1: now also J1.1 (In)
